Commit message: kumi spawn, controllers spawn and com_calculator

File: description/controls.xacro (robot description, xacro)
@@ -42,5 +42,5 @@
     </ros2_control>
     <gazebo>
-        <plugin name="gz_ros2_control-system" name="gz_ros2_control::GazeboSimROS2ControlPlugin">
+        <plugin filename="gz_ros2_control-system" name="gz_ros2_control::GazeboSimROS2ControlPlugin">
             <parameters>/home/andreas/dev_ws/install/kumi/share/kumi/config/kumi_effort_cntr_cnfg.yaml</parameters>
         </plugin>

File: description/kumi.xacro (robot description, xacro)
@@ -2,4 +2,5 @@
 <robot xmlns:xacro="http://www.ros.org/wiki/xacro"  name="kumi">
     <xacro:include filename="/home/andreas/dev_ws/src/kumi/description/variables.xacro" />
+    <xacro:include filename="/home/andreas/dev_ws/src/kumi/description/controls.xacro" />
     <xacro:include filename="/home/andreas/dev_ws/src/kumi/description/kumi_core.xacro" />
 </robot>

File: description/kumi_core.xacro (robot description, xacro)
@@ -1,10 +1,4 @@
 <?xml version="1.0" ?>
 <robot xmlns:xacro="http://www.ros.org/wiki/xacro"  name="kumi">
-    <link name="world" />
-    <joint name="world_to_body" type="fixed">
-        <origin xyz="0 0 5" rpy="0 0 0"/>
-        <parent link="world"/>
-        <child link="body"/>
-    </joint>
     <link name="body">
         <visual>
@@ -14,5 +8,5 @@
             </geometry>
             <material name="green">
-                <color rgba="0.2 1 0.2 1"/>
+                <color rgba="1 0 0 1"/>
             </material>
         </visual>
@@ -34,5 +28,5 @@
         <child link="front_leg"/>
         <axis xyz="0 -1 0"/>
-        <limit lower="-0.7" upper="1" velocity="5" effort="6"/>
+        <limit lower="-0.85" upper="${pi - 0.85}" velocity="5" effort="6"/>
         <dynamics damping="0.5" friction="${joint_friction}"/>
     </joint>
@@ -44,5 +38,5 @@
             </geometry>
             <material name="orange">
-                <color rgba="0.2 1 0.2 1"/>
+                <color rgba="0.7 0.7 0 1"/>
             </material>
         </visual>
@@ -74,5 +68,5 @@
             </geometry>
             <material name="orange">
-                <color rgba="0.2 1 0.2 1"/>
+                <color rgba="0.7 0.7 0 1"/>
             </material>
         </visual>
@@ -94,5 +88,5 @@
         <child link="front_foot"/>
         <axis xyz="0 -1 0"/>
-        <limit lower="-0.5" upper="0.5" velocity="5" effort="2"/>
+        <limit lower="-0.85" upper="0.85" velocity="5" effort="2"/>
         <dynamics damping="0.1" friction="${joint_friction}"/>
     </joint>
@@ -104,5 +98,5 @@
             </geometry>
             <material name="white">
-                <color rgba="0.2 1 0.2 1"/>
+                <color rgba="0 0.5 0.8 1"/>
             </material>
         </visual>
@@ -124,5 +118,5 @@
         <child link="back_leg"/>
         <axis xyz="0 -1 0"/>
-        <limit lower="-0.5" upper="0.5" velocity="5" effort="2"/>
+        <limit lower="${-pi + 0.85}" upper="0.85" velocity="5" effort="2"/>
         <dynamics damping="0.1" friction="${joint_friction}"/>
     </joint>
@@ -134,5 +128,5 @@
             </geometry>
             <material name="orange">
-                <color rgba="0.2 1 0.2 1"/>
+                <color rgba="0.7 0.7 0 1"/>
             </material>
         </visual>
@@ -164,5 +158,5 @@
             </geometry>
             <material name="orange">
-                <color rgba="0.2 1 0.2 1"/>
+                <color rgba="0.7 0.7 0 1"/>
             </material>
         </visual>
@@ -184,5 +178,5 @@
         <child link="back_foot"/>
         <axis xyz="0 -1 0"/>
-        <limit lower="-0.5" upper="0.5" velocity="5" effort="2"/>
+        <limit lower="-0.85" upper="0.85" velocity="5" effort="2"/>
         <dynamics damping="0.1" friction="${joint_friction}"/>
     </joint>
@@ -194,5 +188,5 @@
             </geometry>
             <material name="white">
-                <color rgba="0.2 1 0.2 1"/>
+                <color rgba="0 0.5 0.8 1"/>
             </material>
         </visual>

File: description/variables.xacro (robot description, xacro)
@@ -1,4 +1,7 @@
 <?xml version="1.0" ?>
 <robot xmlns:xacro="http://www.ros.org/wiki/xacro"  name="kumi">
+    <xacro:property name="pi" value="3.14159" />
+    <xacro:property name="ang_low_lim" value="0.85" />
+    <xacro:property name="ang_up_lim" value="4" />
     <xacro:property name="thikness" value="0.15" />
     <xacro:property name="lenght" value="0.5" />

Commit message: traj working, new friction

File: description/controls.xacro (robot description, xacro)
@@ -5,36 +5,30 @@
         </hardware>
         <joint name="front_sh">
-            <command_interface name="effort"/>
-            <state_interface name="effort"/>
+            <command_interface name="position"/>
+            <state_interface name="position"/>
+            <state_interface name="velocity"/>
+        </joint>
+        <joint name="front_knee">
+            <command_interface name="position"/>
+            <state_interface name="position"/>
+            <state_interface name="velocity"/>
+        </joint>
+        <joint name="front_ank">
+            <command_interface name="position"/>
             <state_interface name="position"/>
             <state_interface name="velocity"/>
         </joint>
         <joint name="back_sh">
-            <command_interface name="effort"/>
-            <state_interface name="effort"/>
-            <state_interface name="position"/>
-            <state_interface name="velocity"/>
-        </joint>
-        <joint name="front_knee">
-            <command_interface name="effort"/>
-            <state_interface name="effort"/>
+            <command_interface name="position"/>
             <state_interface name="position"/>
             <state_interface name="velocity"/>
         </joint>
         <joint name="back_knee">
-            <command_interface name="effort"/>
-            <state_interface name="effort"/>
-            <state_interface name="position"/>
-            <state_interface name="velocity"/>
-        </joint>
-        <joint name="front_ank">
-            <command_interface name="effort"/>
-            <state_interface name="effort"/>
+            <command_interface name="position"/>
             <state_interface name="position"/>
             <state_interface name="velocity"/>
         </joint>
         <joint name="back_ank">
-            <command_interface name="effort"/>
-            <state_interface name="effort"/>
+            <command_interface name="position"/>
             <state_interface name="position"/>
             <state_interface name="velocity"/>
@@ -43,5 +37,5 @@
     <gazebo>
         <plugin filename="gz_ros2_control-system" name="gz_ros2_control::GazeboSimROS2ControlPlugin">
-            <parameters>/home/andreas/dev_ws/install/kumi/share/kumi/config/kumi_effort_cntr_cnfg.yaml</parameters>
+            <parameters>/home/andreas/dev_ws/install/kumi/share/kumi/config/kumi_control_config.yaml</parameters>
         </plugin>
     </gazebo>

File: description/kumi_core.xacro (robot description, xacro)
@@ -19,5 +19,5 @@
         <inertial>
             <origin xyz="0 0 0" rpy="0 0 0"/>
-            <mass value="0.5" />
+            <mass value="0.4" />
             <inertia ixx="0.001875" ixy="0.0" ixz="0.0" iyy="0.011354" iyz="0.0" izz="0.011354" />
         </inertial>
@@ -49,5 +49,5 @@
         <inertial>
             <origin xyz="0 0 ${-leg_len/2}" rpy="0 0 0"/>
-            <mass value="0.3" />
+            <mass value="0.2" />
             <inertia ixx="0.001562" ixy="0.0" ixz="0.0" iyy="0.001562" iyz="0.0" izz="0.001125" />
         </inertial>
@@ -79,5 +79,5 @@
         <inertial>
             <origin xyz="0 0 0" rpy="0 0 0"/>
-            <mass value="0.3" />
+            <mass value="0.2" />
             <inertia ixx="0.001562" ixy="0.0" ixz="0.0" iyy="0.001562" iyz="0.0" izz="0.001125" />
         </inertial>
@@ -88,5 +88,5 @@
         <child link="front_foot"/>
         <axis xyz="0 -1 0"/>
-        <limit lower="-0.85" upper="0.85" velocity="5" effort="2"/>
+        <limit lower="-0.85" upper="0.85" velocity="5" effort="6"/>
         <dynamics damping="0.1" friction="${joint_friction}"/>
     </joint>
@@ -109,5 +109,5 @@
         <inertial>
             <origin xyz="0 0 0" rpy="0 0 0"/>
-            <mass value="0.2" />
+            <mass value="0.15" />
             <inertia ixx="0.001135" ixy="0.0" ixz="0.0" iyy="0.001135" iyz="0.0" izz="0.002083" />
         </inertial>
@@ -118,5 +118,5 @@
         <child link="back_leg"/>
         <axis xyz="0 -1 0"/>
-        <limit lower="${-pi + 0.85}" upper="0.85" velocity="5" effort="2"/>
+        <limit lower="${-pi + 0.3}" upper="0.3" velocity="5" effort="6"/>
         <dynamics damping="0.1" friction="${joint_friction}"/>
     </joint>
@@ -139,5 +139,5 @@
         <inertial>
             <origin xyz="0 0 ${-leg_len/2}" rpy="0 0 0"/>
-            <mass value="0.3" />
+            <mass value="0.2" />
             <inertia ixx="0.001562" ixy="0.0" ixz="0.0" iyy="0.001562" iyz="0.0" izz="0.001125" />
         </inertial>
@@ -169,5 +169,5 @@
         <inertial>
             <origin xyz="0 0 0" rpy="0 0 0"/>
-            <mass value="0.3" />
+            <mass value="0.2" />
             <inertia ixx="0.001562" ixy="0.0" ixz="0.0" iyy="0.001562" iyz="0.0" izz="0.001125" />
         </inertial>
@@ -178,5 +178,5 @@
         <child link="back_foot"/>
         <axis xyz="0 -1 0"/>
-        <limit lower="-0.85" upper="0.85" velocity="5" effort="2"/>
+        <limit lower="-0.85" upper="0.85" velocity="5" effort="6"/>
         <dynamics damping="0.1" friction="${joint_friction}"/>
     </joint>
@@ -199,5 +199,5 @@
         <inertial>
             <origin xyz="0 0 0" rpy="0 0 0"/>
-            <mass value="0.2" />
+            <mass value="0.15" />
             <inertia ixx="0.001135" ixy="0.0" ixz="0.0" iyy="0.001135" iyz="0.0" izz="0.002083" />
         </inertial>

File: description/variables.xacro (robot description, xacro)
@@ -7,7 +7,7 @@
     <xacro:property name="lenght" value="0.5" />
     <xacro:property name="leg_len" value="0.4" />
-    <xacro:property name="foot_len" value="0.25" />
+    <xacro:property name="foot_len" value="0.5" />
     <xacro:property name="toll" value="0.005" />
     <xacro:property name="mass" value="0.3" />
-    <xacro:property name="joint_friction" value="0.5" />
+    <xacro:property name="joint_friction" value="0.2" />
 </robot>
