Commit message: setup di Foxglove per visualizzazione dati, da finire di sistemare PID_tuner_GUI e il controllore in quanto si mescolano ancora i dati, introdotto modello di kumi fluttuante con body fisso per tuning pid

File: description/kumi.xacro (robot description, xacro)
@@ -7,5 +7,5 @@
     <xacro:property name="toll" value="0.005" />
     <xacro:property name="mass" value="0.3" />
-    <xacro:property name="joint_friction" value="0.5" />
+    <xacro:property name="joint_friction" value="0.2" />
     <ros2_control name="KumiHardware" type="system">
         <hardware>
@@ -53,5 +53,11 @@
             <parameters>/home/andreas/dev_ws/install/kumi/share/kumi/config/kumi_effort_cntr_cnfg.yaml</parameters>
         </plugin>
-    </gazebo>s
+    </gazebo>
+    <link name="world" />
+    <joint name="world_to_body" type="fixed">
+        <origin xyz="0 0 5" rpy="0 0 0"/>
+        <parent link="world"/>
+        <child link="body"/>
+    </joint>
     <link name="body">
         <visual>
@@ -81,6 +87,6 @@
         <child link="front_leg"/>
         <axis xyz="0 -1 0"/>
-        <limit lower="-0.5" upper="0.5" velocity="5" effort="2"/>
-        <dynamics damping="0.1" friction="${joint_friction}"/>
+        <limit lower="-0.7" upper="1" velocity="5" effort="6"/>
+        <dynamics damping="0.5" friction="${joint_friction}"/>
     </joint>
     <link name="front_leg">
@@ -111,5 +117,5 @@
         <child link="front_leg_d"/>
         <axis xyz="0 0 1"/>
-        <limit lower="-0.5" upper="0.5" velocity="5" effort="2"/>
+        <limit lower="0.0" upper="0.0" velocity="5" effort="2"/>
         <dynamics damping="10.0" friction="10.0"/>
     </joint>
@@ -201,5 +207,5 @@
         <child link="back_leg_d"/>
         <axis xyz="0 0 1"/>
-        <limit lower="-0.5" upper="0.5" velocity="5" effort="2"/>
+        <limit lower="0.0" upper="0.0" velocity="5" effort="2"/>
         <dynamics damping="10.0" friction="10.0"/>
     </joint>

Commit message: last ros2 humble update

File: description/kumi.xacro (robot description, xacro)
@@ -1,264 +1,6 @@
 <?xml version="1.0" ?>
 <robot xmlns:xacro="http://www.ros.org/wiki/xacro"  name="kumi">
-    <xacro:property name="thikness" value="0.15" />
-    <xacro:property name="lenght" value="0.5" />
-    <xacro:property name="leg_len" value="0.4" />
-    <xacro:property name="foot_len" value="0.25" />
-    <xacro:property name="toll" value="0.005" />
-    <xacro:property name="mass" value="0.3" />
-    <xacro:property name="joint_friction" value="0.2" />
-    <ros2_control name="KumiHardware" type="system">
-        <hardware>
-            <plugin>gazebo_ros2_control/GazeboSystem</plugin>
-        </hardware>
-        <joint name="front_sh">
-            <command_interface name="effort"/>
-            <state_interface name="effort"/>
-            <state_interface name="position"/>
-            <state_interface name="velocity"/>
-        </joint>
-        <joint name="back_sh">
-            <command_interface name="effort"/>
-            <state_interface name="effort"/>
-            <state_interface name="position"/>
-            <state_interface name="velocity"/>
-        </joint>
-        <joint name="front_knee">
-            <command_interface name="effort"/>
-            <state_interface name="effort"/>
-            <state_interface name="position"/>
-            <state_interface name="velocity"/>
-        </joint>
-        <joint name="back_knee">
-            <command_interface name="effort"/>
-            <state_interface name="effort"/>
-            <state_interface name="position"/>
-            <state_interface name="velocity"/>
-        </joint>
-        <joint name="front_ank">
-            <command_interface name="effort"/>
-            <state_interface name="effort"/>
-            <state_interface name="position"/>
-            <state_interface name="velocity"/>
-        </joint>
-        <joint name="back_ank">
-            <command_interface name="effort"/>
-            <state_interface name="effort"/>
-            <state_interface name="position"/>
-            <state_interface name="velocity"/>
-        </joint>
-    </ros2_control>
-    <gazebo>
-        <plugin name="gazebo_ros2_control" filename="libgazebo_ros2_control.so">
-            <parameters>/home/andreas/dev_ws/install/kumi/share/kumi/config/kumi_effort_cntr_cnfg.yaml</parameters>
-        </plugin>
-    </gazebo>
-    <link name="world" />
-    <joint name="world_to_body" type="fixed">
-        <origin xyz="0 0 5" rpy="0 0 0"/>
-        <parent link="world"/>
-        <child link="body"/>
-    </joint>
-    <link name="body">
-        <visual>
-            <origin xyz="0 0 0" rpy="0 0 0"/>
-            <geometry>
-                <box size="${lenght} ${thikness} ${thikness}" />
-            </geometry>
-            <material name="green">
-                <color rgba="0.2 1 0.2 1"/>
-            </material>
-        </visual>
-        <collision>
-            <origin xyz="0 0 0" rpy="0 0 0"/>
-            <geometry>
-                <box size="${lenght-toll} ${thikness-toll} ${thikness-toll}" />
-            </geometry>
-        </collision>
-        <inertial>
-            <origin xyz="0 0 0" rpy="0 0 0"/>
-            <mass value="0.5" />
-            <inertia ixx="0.001875" ixy="0.0" ixz="0.0" iyy="0.011354" iyz="0.0" izz="0.011354" />
-        </inertial>
-    </link>
-   <joint name="front_sh" type="revolute">
-        <origin xyz="${lenght} 0 0" rpy="0 0 0"/>
-        <parent link="body"/>
-        <child link="front_leg"/>
-        <axis xyz="0 -1 0"/>
-        <limit lower="-0.7" upper="1" velocity="5" effort="6"/>
-        <dynamics damping="0.5" friction="${joint_friction}"/>
-    </joint>
-    <link name="front_leg">
-        <visual>
-            <origin xyz="0 0 ${-leg_len/2}" rpy="0 0 0"/>
-            <geometry>
-                <box size="${thikness} ${thikness} ${leg_len/2}" />
-            </geometry>
-            <material name="orange">
-                <color rgba="0.2 1 0.2 1"/>
-            </material>
-        </visual>
-        <collision>
-            <origin xyz="0 0 ${-leg_len/2}" rpy="0 0 0"/>
-            <geometry>
-                <box size="${thikness-toll} ${thikness-toll} ${leg_len/2-toll}" />
-            </geometry>
-        </collision>
-        <inertial>
-            <origin xyz="0 0 ${-leg_len/2}" rpy="0 0 0"/>
-            <mass value="0.3" />
-            <inertia ixx="0.001562" ixy="0.0" ixz="0.0" iyy="0.001562" iyz="0.0" izz="0.001125" />
-        </inertial>
-    </link>
-    <joint name="front_knee" type="revolute">
-        <origin xyz="0 0 ${-leg_len}" rpy="0 0 0"/>
-        <parent link="front_leg"/>
-        <child link="front_leg_d"/>
-        <axis xyz="0 0 1"/>
-        <limit lower="0.0" upper="0.0" velocity="5" effort="2"/>
-        <dynamics damping="10.0" friction="10.0"/>
-    </joint>
-    <link name="front_leg_d">
-        <visual>
-            <origin xyz="0 0 0" rpy="0 0 0"/>
-            <geometry>
-                <box size="${thikness} ${thikness} ${leg_len/2}" />
-            </geometry>
-            <material name="orange">
-                <color rgba="0.2 1 0.2 1"/>
-            </material>
-        </visual>
-        <collision>
-            <origin xyz="0 0 0" rpy="0 0 0"/>
-            <geometry>
-                <box size="${thikness-toll} ${thikness-toll} ${leg_len/2-toll}" />
-            </geometry>
-        </collision>
-        <inertial>
-            <origin xyz="0 0 0" rpy="0 0 0"/>
-            <mass value="0.3" />
-            <inertia ixx="0.001562" ixy="0.0" ixz="0.0" iyy="0.001562" iyz="0.0" izz="0.001125" />
-        </inertial>
-    </link>
-    <joint name="front_ank" type="revolute">
-        <origin xyz="0 0 ${-leg_len/2 - thikness/2}" rpy="0 0 0"/>
-        <parent link="front_leg_d"/>
-        <child link="front_foot"/>
-        <axis xyz="0 -1 0"/>
-        <limit lower="-0.5" upper="0.5" velocity="5" effort="2"/>
-        <dynamics damping="0.1" friction="${joint_friction}"/>
-    </joint>
-    <link name="front_foot">
-        <visual>
-            <origin xyz="0 0 0" rpy="0 0 0"/>
-            <geometry>
-                <box size="${foot_len} ${foot_len} ${thikness/2}" />
-            </geometry>
-            <material name="white">
-                <color rgba="0.2 1 0.2 1"/>
-            </material>
-        </visual>
-        <collision>
-            <origin xyz="0 0 0" rpy="0 0 0"/>
-            <geometry>
-                <box size="${foot_len-toll} ${foot_len-toll} ${thikness/2-toll}" />
-            </geometry>
-        </collision>
-        <inertial>
-            <origin xyz="0 0 0" rpy="0 0 0"/>
-            <mass value="0.2" />
-            <inertia ixx="0.001135" ixy="0.0" ixz="0.0" iyy="0.001135" iyz="0.0" izz="0.002083" />
-        </inertial>
-    </link>
-    <joint name="back_sh" type="revolute">
-        <origin xyz="${-lenght} 0 0" rpy="0 0 0"/>
-        <parent link="body"/>
-        <child link="back_leg"/>
-        <axis xyz="0 -1 0"/>
-        <limit lower="-0.5" upper="0.5" velocity="5" effort="2"/>
-        <dynamics damping="0.1" friction="${joint_friction}"/>
-    </joint>
-    <link name="back_leg">
-        <visual>
-            <origin xyz="0 0 ${-leg_len/2}" rpy="0 0 0"/>
-            <geometry>
-                <box size="${thikness} ${thikness} ${leg_len/2}" />
-            </geometry>
-            <material name="orange">
-                <color rgba="0.2 1 0.2 1"/>
-            </material>
-        </visual>
-        <collision>
-            <origin xyz="0 0 ${-leg_len/2}" rpy="0 0 0"/>
-            <geometry>
-                <box size="${thikness-toll} ${thikness-toll} ${leg_len/2-toll}" />
-            </geometry>
-        </collision>
-        <inertial>
-            <origin xyz="0 0 ${-leg_len/2}" rpy="0 0 0"/>
-            <mass value="0.3" />
-            <inertia ixx="0.001562" ixy="0.0" ixz="0.0" iyy="0.001562" iyz="0.0" izz="0.001125" />
-        </inertial>
-    </link>
-    <joint name="back_knee" type="revolute">
-        <origin xyz="0 0 ${-leg_len}" rpy="0 0 0"/>
-        <parent link="back_leg"/>
-        <child link="back_leg_d"/>
-        <axis xyz="0 0 1"/>
-        <limit lower="0.0" upper="0.0" velocity="5" effort="2"/>
-        <dynamics damping="10.0" friction="10.0"/>
-    </joint>
-    <link name="back_leg_d">
-        <visual>
-            <origin xyz="0 0 0" rpy="0 0 0"/>
-            <geometry>
-                <box size="${thikness} ${thikness} ${leg_len/2}" />
-            </geometry>
-            <material name="orange">
-                <color rgba="0.2 1 0.2 1"/>
-            </material>
-        </visual>
-        <collision>
-            <origin xyz="0 0 0" rpy="0 0 0"/>
-            <geometry>
-                <box size="${thikness-toll} ${thikness-toll} ${leg_len/2-toll}" />
-            </geometry>
-        </collision>
-        <inertial>
-            <origin xyz="0 0 0" rpy="0 0 0"/>
-            <mass value="0.3" />
-            <inertia ixx="0.001562" ixy="0.0" ixz="0.0" iyy="0.001562" iyz="0.0" izz="0.001125" />
-        </inertial>
-    </link>
-    <joint name="back_ank" type="revolute">
-        <origin xyz="0 0 ${-leg_len/2 - thikness/2}" rpy="0 0 0"/>
-        <parent link="back_leg_d"/>
-        <child link="back_foot"/>
-        <axis xyz="0 -1 0"/>
-        <limit lower="-0.5" upper="0.5" velocity="5" effort="2"/>
-        <dynamics damping="0.1" friction="${joint_friction}"/>
-    </joint>
-    <link name="back_foot">
-        <visual>
-            <origin xyz="0 0 0" rpy="0 0 0"/>
-            <geometry>
-                <box size="${foot_len} ${foot_len} ${thikness/2}" />
-            </geometry>
-            <material name="white">
-                <color rgba="0.2 1 0.2 1"/>
-            </material>
-        </visual>
-        <collision>
-            <origin xyz="0 0 0" rpy="0 0 0"/>
-            <geometry>
-                <box size="${foot_len-toll} ${foot_len-toll} ${thikness/2-toll}" />
-            </geometry>
-        </collision>
-        <inertial>
-            <origin xyz="0 0 0" rpy="0 0 0"/>
-            <mass value="0.2" />
-            <inertia ixx="0.001135" ixy="0.0" ixz="0.0" iyy="0.001135" iyz="0.0" izz="0.002083" />
-        </inertial>
-    </link>
+    <xacro:include filename="/home/andreas/dev_ws/src/kumi/description/variables.xacro" />
+    <xacro:include filename="/home/andreas/dev_ws/src/kumi/description/controls.xacro" />
+    <xacro:include filename="/home/andreas/dev_ws/src/kumi/description/kumi_core.xacro" />
 </robot>
