Commit message: last ros2 humble update

File: description/kumi_core.xacro (robot description, xacro)
@@ -1,64 +1,15 @@
-<robot xmlns:xacro="http://www.ros.org/wiki/xacro"  name="robot">
-    <xacro:property name="thikness" value="0.15" />
-    <xacro:property name="lenght" value="0.5" />
-    <xacro:property name="leg_len" value="0.5" />
-    <xacro:property name="foot_len" value="0.2" />
-    <xacro:property name="toll" value="0.005" />
-    <xacro:property name="mass" value="0.3" />
-    <ros2_control name="KumiHardware" type="system">
-        <hardware>
-            <plugin>gazebo_ros2_control/GazeboSystem</plugin>
-        </hardware>
-        <joint name="front_sh">
-            <command_interface name="position"/>
-            <state_interface name="position"/>
-            <state_interface name="velocity"/>
-        </joint>
-        <joint name="back_sh">
-            <command_interface name="position"/>
-            <state_interface name="position"/>
-            <state_interface name="velocity"/>
-        </joint>
-        <joint name="front_knee">
-            <command_interface name="position"/>
-            <state_interface name="position"/>
-            <state_interface name="velocity"/>
-        </joint>
-        <joint name="back_knee">
-            <command_interface name="position"/>
-            <state_interface name="position"/>
-            <state_interface name="velocity"/>
-        </joint>
-        <joint name="front_ank">
-            <command_interface name="position"/>
-            <state_interface name="position"/>
-            <state_interface name="velocity"/>
-        </joint>
-        <joint name="back_ank">
-            <command_interface name="position"/>
-            <state_interface name="position"/>
-            <state_interface name="velocity"/>
-        </joint>
-    </ros2_control>
-    <gazebo>
-        <plugin name="gazebo_ros2_control" filename="libgazebo_ros2_control.so">
-            <parameters>/home/andreas/dev_ws/install/kumi_controller/share/kumi_controller/config/kumi_effort_cntr_cnfg.yaml</parameters>
-        </plugin>
-    </gazebo>
-    <physics type="ode">
-    <max_step_size>0.001</max_step_size>
-    <real_time_update_rate>1000</real_time_update_rate>
-    <ode>
-        <solver>
-        <iters>50</iters>
-        <sor>1.3</sor>
-        </solver>
-    </ode>
-    </physics>
+<?xml version="1.0" ?>
+<robot xmlns:xacro="http://www.ros.org/wiki/xacro"  name="kumi">
+    <link name="world" />
+    <joint name="world_to_body" type="fixed">
+        <origin xyz="0 0 5" rpy="0 0 0"/>
+        <parent link="world"/>
+        <child link="body"/>
+    </joint>
     <link name="body">
         <visual>
             <origin xyz="0 0 0" rpy="0 0 0"/>
             <geometry>
-                <box size="${lenght+2*thikness} ${thikness*2} ${thikness}" />
+                <box size="${lenght} ${thikness} ${thikness}" />
             </geometry>
             <material name="green">
@@ -69,5 +20,5 @@
             <origin xyz="0 0 0" rpy="0 0 0"/>
             <geometry>
-                <box size="${lenght/1.5-toll} ${thikness*2-toll} ${thikness-toll}" />
+                <box size="${lenght-toll} ${thikness-toll} ${thikness-toll}" />
             </geometry>
         </collision>
@@ -75,101 +26,65 @@
             <origin xyz="0 0 0" rpy="0 0 0"/>
             <mass value="0.5" />
-            <inertia ixx="0.015" ixy="0.0" ixz="0.0" iyy="0.340833" iyz="0.0" izz="0.340833" />
-        </inertial>
-    </link>
-    <gazebo reference="body">
-        <sensor name="imu_sensor" type="imu">
-            <update_rate>20.0</update_rate>
-            <always_on>true</always_on>
-            <imu>
-            <angular_velocity>
-                <noise type="gaussian">
-                <mean>0.0</mean>
-                <stddev>0.1</stddev>
-                </noise>
-            </angular_velocity>
-            <linear_acceleration>
-                <noise type="gaussian">
-                <mean>0.0</mean>
-                <stddev>0.1</stddev>
-                </noise>
-            </linear_acceleration>
-            </imu>
-            <plugin filename="libgazebo_ros_imu_sensor.so" name="imu_sensor">
-            <ros>
-                <namespace>/</namespace>
-                <remapping>~/out:=/imu</remapping>
-            </ros>
-            </plugin>
-        </sensor>
-    </gazebo>
-    <joint name="front_sh" type="revolute">
-        <origin xyz="${lenght/2+thikness/2} 0 0" rpy="0 0 0"/>
+            <inertia ixx="0.001875" ixy="0.0" ixz="0.0" iyy="0.011354" iyz="0.0" izz="0.011354" />
+        </inertial>
+    </link>
+   <joint name="front_sh" type="revolute">
+        <origin xyz="${lenght} 0 0" rpy="0 0 0"/>
         <parent link="body"/>
         <child link="front_leg"/>
         <axis xyz="0 -1 0"/>
-        <limit lower="-${pi/2}" upper="${pi}" velocity="100" effort="100"/>
-    </joint>
-    <transmission name="front_sh_trans">
-        <type>transmission_interface/SimpleTransmission</type>
-        <actuator name="motor1">
-            <mechanicalReduction>1.0</mechanicalReduction>
-        </actuator>
-    </transmission>
+        <limit lower="-0.7" upper="1" velocity="5" effort="6"/>
+        <dynamics damping="0.5" friction="${joint_friction}"/>
+    </joint>
     <link name="front_leg">
         <visual>
-            <origin xyz="0 0 ${-leg_len/4 -thikness/2}" rpy="0 0 0"/>
-            <geometry>
-                <box size="${thikness} ${thikness*2} ${leg_len/2}" />
-            </geometry>
-            <material name="orange">
-                <color rgba="0.2 1 0.2 1"/>
-            </material>
-        </visual>
-        <collision>
-            <origin xyz="0 0 ${-leg_len/4 -thikness/2}" rpy="0 0 0"/>
-            <geometry>
-                <box size="${thikness-toll} ${thikness*2-toll} ${leg_len/2-toll}" />
-            </geometry>
-        </collision>
-        <inertial>
-            <origin xyz="${thikness/2} 0 ${-leg_len/4}" rpy="0 0 0"/>
-            <mass value="0.3" />
-            <inertia ixx="0.090833" ixy="0.0" ixz="0.0" iyy="0.090833" iyz="0.0" izz="0.015000" />
+            <origin xyz="0 0 ${-leg_len/2}" rpy="0 0 0"/>
+            <geometry>
+                <box size="${thikness} ${thikness} ${leg_len/2}" />
+            </geometry>
+            <material name="orange">
+                <color rgba="0.2 1 0.2 1"/>
+            </material>
+        </visual>
+        <collision>
+            <origin xyz="0 0 ${-leg_len/2}" rpy="0 0 0"/>
+            <geometry>
+                <box size="${thikness-toll} ${thikness-toll} ${leg_len/2-toll}" />
+            </geometry>
+        </collision>
+        <inertial>
+            <origin xyz="0 0 ${-leg_len/2}" rpy="0 0 0"/>
+            <mass value="0.3" />
+            <inertia ixx="0.001562" ixy="0.0" ixz="0.0" iyy="0.001562" iyz="0.0" izz="0.001125" />
         </inertial>
     </link>
     <joint name="front_knee" type="revolute">
-        <origin xyz="0 0 ${-leg_len/2-thikness/2}" rpy="0 0 0"/>
+        <origin xyz="0 0 ${-leg_len}" rpy="0 0 0"/>
         <parent link="front_leg"/>
         <child link="front_leg_d"/>
         <axis xyz="0 0 1"/>
-        <limit lower="${-pi/4}" upper="${pi/4}" velocity="100" effort="100"/>
-    </joint>
-    <transmission name="front_knee_trans">
-        <type>transmission_interface/SimpleTransmission</type>
-        <actuator name="motor2">
-            <mechanicalReduction>1.0</mechanicalReduction>
-        </actuator>
-    </transmission>
+        <limit lower="0.0" upper="0.0" velocity="5" effort="2"/>
+        <dynamics damping="10.0" friction="10.0"/>
+    </joint>
     <link name="front_leg_d">
         <visual>
-            <origin xyz="0 0 ${-leg_len/4}" rpy="0 0 0"/>
-            <geometry>
-                <box size="${thikness} ${thikness*2} ${leg_len/2}" />
-            </geometry>
-            <material name="orange">
-                <color rgba="0.2 1 0.2 1"/>
-            </material>
-        </visual>
-        <collision>
-            <origin xyz="0 0 ${-leg_len/4}" rpy="0 0 0"/>
-            <geometry>
-                <box size="${thikness-toll} ${thikness*2-toll} ${leg_len/3-toll}" />
-            </geometry>
-        </collision>
-        <inertial>
-            <origin xyz="0 0 ${-leg_len/4}" rpy="0 0 0"/>
-            <mass value="0.3" />
-            <inertia ixx="0.090833" ixy="0.0" ixz="0.0" iyy="0.090833" iyz="0.0" izz="0.015000" />
+            <origin xyz="0 0 0" rpy="0 0 0"/>
+            <geometry>
+                <box size="${thikness} ${thikness} ${leg_len/2}" />
+            </geometry>
+            <material name="orange">
+                <color rgba="0.2 1 0.2 1"/>
+            </material>
+        </visual>
+        <collision>
+            <origin xyz="0 0 0" rpy="0 0 0"/>
+            <geometry>
+                <box size="${thikness-toll} ${thikness-toll} ${leg_len/2-toll}" />
+            </geometry>
+        </collision>
+        <inertial>
+            <origin xyz="0 0 0" rpy="0 0 0"/>
+            <mass value="0.3" />
+            <inertia ixx="0.001562" ixy="0.0" ixz="0.0" iyy="0.001562" iyz="0.0" izz="0.001125" />
         </inertial>
     </link>
@@ -179,17 +94,12 @@
         <child link="front_foot"/>
         <axis xyz="0 -1 0"/>
-        <limit lower="${-pi/4}" upper="${pi/4}" velocity="100" effort="100"/>
-    </joint>
-    <transmission name="front_ank_trans">
-        <type>transmission_interface/SimpleTransmission</type>
-        <actuator name="motor3">
-            <mechanicalReduction>1.0</mechanicalReduction>
-        </actuator>
-    </transmission>0.0
+        <limit lower="-0.5" upper="0.5" velocity="5" effort="2"/>
+        <dynamics damping="0.1" friction="${joint_friction}"/>
+    </joint>
     <link name="front_foot">
         <visual>
             <origin xyz="0 0 0" rpy="0 0 0"/>
             <geometry>
-                <box size="${foot_len+thikness} ${foot_len*2.5} ${thikness-toll}" />
+                <box size="${foot_len} ${foot_len} ${thikness/2}" />
             </geometry>
             <material name="white">
@@ -200,5 +110,5 @@
             <origin xyz="0 0 0" rpy="0 0 0"/>
             <geometry>
-                <box size="${foot_len+thikness} ${foot_len*2.5} ${thikness-toll}" />
+                <box size="${foot_len-toll} ${foot_len-toll} ${thikness/2-toll}" />
             </geometry>
         </collision>
@@ -206,75 +116,65 @@
             <origin xyz="0 0 0" rpy="0 0 0"/>
             <mass value="0.2" />
-            <inertia ixx="0.241667" ixy="0.0" ixz="0.0" iyy="0.454167" iyz="0.0" izz="0.163333" />
+            <inertia ixx="0.001135" ixy="0.0" ixz="0.0" iyy="0.001135" iyz="0.0" izz="0.002083" />
         </inertial>
     </link>
     <joint name="back_sh" type="revolute">
-        <origin xyz="${-lenght/2-thikness/2} 0 0" rpy="0 0 0"/>
+        <origin xyz="${-lenght} 0 0" rpy="0 0 0"/>
         <parent link="body"/>
         <child link="back_leg"/>
         <axis xyz="0 -1 0"/>
-        <limit lower="-${1.5*pi}" upper="${pi/2}" velocity="100" effort="100"/>
-    </joint>
-    <transmission name="back_sh_trans">
-        <type>transmission_interface/SimpleTransmission</type>
-        <actuator name="motor4">
-            <mechanicalReduction>1.0</mechanicalReduction>
-        </actuator>
-    </transmission>
+        <limit lower="-0.5" upper="0.5" velocity="5" effort="2"/>
+        <dynamics damping="0.1" friction="${joint_friction}"/>
+    </joint>
     <link name="back_leg">
         <visual>
-            <origin xyz="0 0 ${-leg_len/4 -thikness/2}" rpy="0 0 0"/>
-            <geometry>
-                <box size="${thikness} ${thikness*2} ${leg_len/2}" />
-            </geometry>
-            <material name="orange">
-                <color rgba="0.2 1 0.2 1"/>
-            </material>
-        </visual>
-        <collision>
-            <origin xyz="0 0 ${-leg_len/4 -thikness/2}" rpy="0 0 0"/>
-            <geometry>
-                <box size="${thikness-toll} ${thikness*2-toll} ${leg_len/2-toll}" />
-            </geometry>
-        </collision>
-        <inertial>
-            <origin xyz="${-thikness/2} 0 ${-leg_len/4}" rpy="0 0 0"/>
-            <mass value="0.3" />
-            <inertia ixx="0.090833" ixy="0.0" ixz="0.0" iyy="0.090833" iyz="0.0" izz="0.015000" />
+            <origin xyz="0 0 ${-leg_len/2}" rpy="0 0 0"/>
+            <geometry>
+                <box size="${thikness} ${thikness} ${leg_len/2}" />
+            </geometry>
+            <material name="orange">
+                <color rgba="0.2 1 0.2 1"/>
+            </material>
+        </visual>
+        <collision>
+            <origin xyz="0 0 ${-leg_len/2}" rpy="0 0 0"/>
+            <geometry>
+                <box size="${thikness-toll} ${thikness-toll} ${leg_len/2-toll}" />
+            </geometry>
+        </collision>
+        <inertial>
+            <origin xyz="0 0 ${-leg_len/2}" rpy="0 0 0"/>
+            <mass value="0.3" />
+            <inertia ixx="0.001562" ixy="0.0" ixz="0.0" iyy="0.001562" iyz="0.0" izz="0.001125" />
         </inertial>
     </link>
     <joint name="back_knee" type="revolute">
-        <origin xyz="0 0 ${-leg_len/2 -thikness/2}" rpy="0 0 0"/>
+        <origin xyz="0 0 ${-leg_len}" rpy="0 0 0"/>
         <parent link="back_leg"/>
         <child link="back_leg_d"/>
         <axis xyz="0 0 1"/>
-        <limit lower="-${pi/4}" upper="${pi/4}" velocity="100" effort="100"/>
-    </joint>
-    <transmission name="back_knee_trans">
-        <type>transmission_interface/SimpleTransmission</type>
-        <actuator name="motor5">
-            <mechanicalReduction>1.0</mechanicalReduction>
-        </actuator>
-    </transmission>
+        <limit lower="0.0" upper="0.0" velocity="5" effort="2"/>
+        <dynamics damping="10.0" friction="10.0"/>
+    </joint>
     <link name="back_leg_d">
         <visual>
-            <origin xyz="0 0 ${-leg_len/4}" rpy="0 0 0"/>
-            <geometry>
-                <box size="${thikness} ${thikness*2} ${leg_len/2}" />
-            </geometry>
-            <material name="orange">
-                <color rgba="0.2 1 0.2 1"/>
-            </material>
-        </visual>
-        <collision>
-            <origin xyz="0 0 ${-leg_len/4}" rpy="0 0 0"/>
-            <geometry>
-                <box size="${thikness-toll} ${thikness*2-toll} ${leg_len/3-toll}" />
-            </geometry>
-        </collision>
-        <inertial>
-            <origin xyz="0 0 ${-leg_len/4}" rpy="0 0 0"/>
-            <mass value="0.3" />
-            <inertia ixx="0.090833" ixy="0.0" ixz="0.0" iyy="0.090833" iyz="0.0" izz="0.015000" />
+            <origin xyz="0 0 0" rpy="0 0 0"/>
+            <geometry>
+                <box size="${thikness} ${thikness} ${leg_len/2}" />
+            </geometry>
+            <material name="orange">
+                <color rgba="0.2 1 0.2 1"/>
+            </material>
+        </visual>
+        <collision>
+            <origin xyz="0 0 0" rpy="0 0 0"/>
+            <geometry>
+                <box size="${thikness-toll} ${thikness-toll} ${leg_len/2-toll}" />
+            </geometry>
+        </collision>
+        <inertial>
+            <origin xyz="0 0 0" rpy="0 0 0"/>
+            <mass value="0.3" />
+            <inertia ixx="0.001562" ixy="0.0" ixz="0.0" iyy="0.001562" iyz="0.0" izz="0.001125" />
         </inertial>
     </link>
@@ -284,17 +184,12 @@
         <child link="back_foot"/>
         <axis xyz="0 -1 0"/>
-        <limit lower="-${pi/4}" upper="${pi/4}" velocity="100" effort="100"/>
-    </joint>
-    <transmission name="back_ank_trans">
-        <type>transmission_interface/SimpleTransmission</type>
-        <actuator name="motor6">
-            <mechanicalReduction>1.0</mechanicalReduction>
-        </actuator>
-    </transmission>
+        <limit lower="-0.5" upper="0.5" velocity="5" effort="2"/>
+        <dynamics damping="0.1" friction="${joint_friction}"/>
+    </joint>
     <link name="back_foot">
         <visual>
             <origin xyz="0 0 0" rpy="0 0 0"/>
             <geometry>
-                <box size="${foot_len+thikness} ${foot_len*2.5} ${thikness-toll}" />
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