Commit message: added a front and rear camera mounted on the body, changed term back with rear. TODO: camera adgust direction using imu data

File: description/kumi.xacro (robot description, xacro)
@@ -4,3 +4,4 @@
     <xacro:include filename="/home/andreas/dev_ws/src/kumi/description/xacro/effort_control.xacro" />
     <xacro:include filename="/home/andreas/dev_ws/src/kumi/description/xacro/kumi_mesh.xacro" />
+    <xacro:include filename="/home/andreas/dev_ws/src/kumi/description/xacro/cameras_config.xacro" />
 </robot>

File: description/xacro/effort_control.xacro (robot description, xacro)
@@ -16,5 +16,5 @@
             <state_interface name="effort"/>
         </joint>
-        <joint name="back_sh">
+        <joint name="rear_sh">
             <command_interface name="effort"/>
             <state_interface name="position"/>
@@ -22,5 +22,5 @@
             <state_interface name="effort"/>
         </joint>
-        <joint name="back_ank">
+        <joint name="rear_ank">
             <command_interface name="effort"/>
             <state_interface name="position"/>

File: description/xacro/kumi_core.xacro (robot description, xacro)
@@ -113,73 +113,73 @@
         </inertial>
     </link>
-    <joint name="back_sh" type="revolute">
+    <joint name="rear_sh" type="revolute">
         <origin xyz="${-lenght} 0 0" rpy="0 0 0"/>
         <parent link="body"/>
-        <child link="back_leg"/>
+        <child link="rear_leg"/>
         <axis xyz="0 1 0"/>
         <limit lower="${-pi + 0.3}" upper="0.3" velocity="5" effort="6"/>
         <dynamics damping="0.1" friction="${joint_friction}"/>
     </joint>
-    <link name="back_leg">
-        <visual>
-            <origin xyz="0 0 ${-leg_len/2}" rpy="0 0 0"/>
-            <geometry>
-                <box size="${thikness} ${thikness} ${leg_len/2}" />
-            </geometry>
-            <material name="orange">
-                <color rgba="0.7 0.7 0 1"/>
-            </material>
-        </visual>
-        <collision>
-            <origin xyz="0 0 ${-leg_len/2}" rpy="0 0 0"/>
-            <geometry>
-                <box size="${thikness-toll} ${thikness-toll} ${leg_len/2-toll}" />
-            </geometry>
-        </collision>
-        <inertial>
-            <origin xyz="0 0 ${-leg_len/2}" rpy="0 0 0"/>
-            <mass value="0.2" />
-            <inertia ixx="0.001562" ixy="0.0" ixz="0.0" iyy="0.001562" iyz="0.0" izz="0.001125" />
-        </inertial>
-    </link>
-    <joint name="back_knee" type="revolute">
+    <link name="rear_leg">
+        <visual>
+            <origin xyz="0 0 ${-leg_len/2}" rpy="0 0 0"/>
+            <geometry>
+                <box size="${thikness} ${thikness} ${leg_len/2}" />
+            </geometry>
+            <material name="orange">
+                <color rgba="0.7 0.7 0 1"/>
+            </material>
+        </visual>
+        <collision>
+            <origin xyz="0 0 ${-leg_len/2}" rpy="0 0 0"/>
+            <geometry>
+                <box size="${thikness-toll} ${thikness-toll} ${leg_len/2-toll}" />
+            </geometry>
+        </collision>
+        <inertial>
+            <origin xyz="0 0 ${-leg_len/2}" rpy="0 0 0"/>
+            <mass value="0.2" />
+            <inertia ixx="0.001562" ixy="0.0" ixz="0.0" iyy="0.001562" iyz="0.0" izz="0.001125" />
+        </inertial>
+    </link>
+    <joint name="rear_knee" type="revolute">
         <origin xyz="0 0 ${-leg_len}" rpy="0 0 0"/>
-        <parent link="back_leg"/>
-        <child link="back_leg_d"/>
+        <parent link="rear_leg"/>
+        <child link="rear_leg_d"/>
         <axis xyz="0 0 1"/>
         <limit lower="0.0" upper="0.0" velocity="5" effort="2"/>
         <dynamics damping="10.0" friction="10.0"/>
     </joint>
-    <link name="back_leg_d">
-        <visual>
-            <origin xyz="0 0 0" rpy="0 0 0"/>
-            <geometry>
-                <box size="${thikness} ${thikness} ${leg_len/2}" />
-            </geometry>
-            <material name="orange">
-                <color rgba="0.7 0.7 0 1"/>
-            </material>
-        </visual>
-        <collision>
-            <origin xyz="0 0 0" rpy="0 0 0"/>
-            <geometry>
-                <box size="${thikness-toll} ${thikness-toll} ${leg_len/2-toll}" />
-            </geometry>
-        </collision>
-        <inertial>
-            <origin xyz="0 0 0" rpy="0 0 0"/>
-            <mass value="0.2" />
-            <inertia ixx="0.001562" ixy="0.0" ixz="0.0" iyy="0.001562" iyz="0.0" izz="0.001125" />
-        </inertial>
-    </link>
-    <joint name="back_ank" type="revolute">
+    <link name="rear_leg_d">
+        <visual>
+            <origin xyz="0 0 0" rpy="0 0 0"/>
+            <geometry>
+                <box size="${thikness} ${thikness} ${leg_len/2}" />
+            </geometry>
+            <material name="orange">
+                <color rgba="0.7 0.7 0 1"/>
+            </material>
+        </visual>
+        <collision>
+            <origin xyz="0 0 0" rpy="0 0 0"/>
+            <geometry>
+                <box size="${thikness-toll} ${thikness-toll} ${leg_len/2-toll}" />
+            </geometry>
+        </collision>
+        <inertial>
+            <origin xyz="0 0 0" rpy="0 0 0"/>
+            <mass value="0.2" />
+            <inertia ixx="0.001562" ixy="0.0" ixz="0.0" iyy="0.001562" iyz="0.0" izz="0.001125" />
+        </inertial>
+    </link>
+    <joint name="rear_ank" type="revolute">
         <origin xyz="0 0 ${-leg_len/4 - thikness/4}" rpy="0 0 0"/>
-        <parent link="back_leg_d"/>
-        <child link="back_foot"/>
+        <parent link="rear_leg_d"/>
+        <child link="rear_foot"/>
         <axis xyz="0 1 0"/>
         <limit lower="-0.85" upper="0.85" velocity="5" effort="6"/>
         <dynamics damping="0.1" friction="${joint_friction}"/>
     </joint>
-    <link name="back_foot">
+    <link name="rear_foot">
         <visual>
             <origin xyz="0 0 ${-leg_len/4 - thikness/4}" rpy="0 0 0"/>

File: description/xacro/kumi_mesh_old.xacro (robot description, xacro)
@@ -25,26 +25,4 @@
             <mass value="0.15"/>
             <inertia ixx="0.000226" ixy="0.0" ixz="0.0" iyy="0.000755" iyz="0.0" izz="0.000971"/>
-        </inertial>
-    </link>
-    <joint name="front_camera_joint" type="fixed">
-        <parent link="body"/>
-        <child link="front_camera"/>
-        <origin xyz="-0.105 -0.03 0.0" rpy="0 0 ${pi}"/>
-        <axis xyz="0 0 1"/>
-    </joint>
-    <link name="front_camera">
-        <visual>
-            <origin xyz="0 0 0" rpy="0 0 0"/>
-            <geometry>
-                <box size="0.01 0.01 0.01"/>
-            </geometry>
-            <material name="gray">
-                <color rgba="0 0 0 0.8"/>
-            </material>
-        </visual>
-        <inertial>
-            <origin xyz="0 0 0" rpy="0 0 0"/>
-            <mass value="0.035"/>
-            <inertia ixx="0.001" ixy="0.0" ixz="0.0" iyy="0.001" iyz="0.0" izz="0.001"/>
         </inertial>
     </link>
@@ -127,26 +105,4 @@
             <mass value="0.15"/>
             <inertia ixx="0.000091" ixy="0.0" ixz="0.0" iyy="0.000165" iyz="0.0" izz="0.000091"/>
-        </inertial>
-    </link>
-    <joint name="rear_camera_joint" type="fixed">
-        <parent link="body"/>
-        <child link="rear_camera"/>
-        <origin xyz="0.105 0.03 0.0" rpy="0 0 0"/>
-        <axis xyz="0 0 1"/>
-    </joint>
-    <link name="rear_camera">
-        <visual>
-            <origin xyz="0 0 0" rpy="0 0 0"/>
-            <geometry>
-                <box size="0.01 0.01 0.01"/>
-            </geometry>
-            <material name="gray">
-                <color rgba="0 0 0 0.8"/>
-            </material>
-        </visual>
-        <inertial>
-            <origin xyz="0 0 0" rpy="0 0 0"/>
-            <mass value="0.035"/>
-            <inertia ixx="0.001" ixy="0.0" ixz="0.0" iyy="0.001" iyz="0.0" izz="0.001"/>
         </inertial>
     </link>

File: description/xacro/trajectory_control.xacro (robot description, xacro)
@@ -14,10 +14,10 @@
             <state_interface name="velocity"/>
         </joint>
-        <joint name="back_sh">
+        <joint name="rear_sh">
             <command_interface name="position"/>
             <state_interface name="position"/>
             <state_interface name="velocity"/>
         </joint>
-        <joint name="back_ank">
+        <joint name="rear_ank">
             <command_interface name="position"/>
             <state_interface name="position"/>

Commit message: added IMU: working but pose not computed. added contact sensors: not working, maybe i should simplify the geometry of the collision in orther to symplify computation.

File: description/kumi.xacro (robot description, xacro)
@@ -4,4 +4,4 @@
     <xacro:include filename="/home/andreas/dev_ws/src/kumi/description/xacro/effort_control.xacro" />
     <xacro:include filename="/home/andreas/dev_ws/src/kumi/description/xacro/kumi_mesh.xacro" />
-    <xacro:include filename="/home/andreas/dev_ws/src/kumi/description/xacro/cameras_config.xacro" />
+    <xacro:include filename="/home/andreas/dev_ws/src/kumi/description/xacro/sensors_config.xacro" />
 </robot>

File: description/xacro/kumi_mesh.xacro (robot description, xacro)
@@ -117,5 +117,5 @@
             </material>
         </visual>
-        <collision>
+        <collision name="frontFootCollision">
             <origin xyz="0 0 0" rpy="${pi/2} 0  ${-pi/2}"/>
             <geometry>
@@ -219,5 +219,5 @@
             </material>
         </visual>
-        <collision>
+        <collision name="rearFootCollision">
             <origin xyz="0 0 0" rpy="${pi/2} 0  ${pi/2}"/>
             <geometry>

File: description/xacro/sensors_config.xacro (robot description, xacro)
@@ -57,3 +57,42 @@
         </sensor>
     </gazebo>
+    <gazebo reference="body">
+        <sensor name="imu_sensor" type="imu">
+            <always_on>true</always_on>
+            <update_rate>100</update_rate>
+            <topic>/bodyImu/data</topic>
+            <imu>
+                <angular_velocity>
+                    <x noise_type="gaussian" mean="0.0" stddev="0.001"/>
+                    <y noise_type="gaussian" mean="0.0" stddev="0.001"/>
+                    <z noise_type="gaussian" mean="0.0" stddev="0.001"/>
+                </angular_velocity>
+                <linear_acceleration>
+                    <x noise_type="gaussian" mean="0.0" stddev="0.01"/>
+                    <y noise_type="gaussian" mean="0.0" stddev="0.01"/>
+                    <z noise_type="gaussian" mean="0.0" stddev="0.01"/>
+                </linear_acceleration>
+            </imu>
+        </sensor>
+    </gazebo>
+    <gazebo reference="front_foot">
+        <sensor name='frontFootCollision' type='contact'>
+          <contact>
+            <collision>frontFootCollision</collision>
+            <topic>/frontFootCollisionFlag</topic>
+          </contact>
+          <always_on>1</always_on>
+          <update_rate>100</update_rate>
+        </sensor>
+    </gazebo>
+    <gazebo reference="rear_foot">
+        <sensor name='rearFootCollision' type='contact'>
+          <contact>
+            <collision>rearFootCollision</collision>
+            <topic>/rearFootCollisionFlag</topic>
+          </contact>
+          <always_on>1</always_on>
+          <update_rate>100</update_rate>
+        </sensor>
+    </gazebo>
 </robot>

Commit message: absolute paths changed with relative paths

File: description/kumi.xacro (robot description, xacro)
@@ -1,7 +1,8 @@
 <?xml version="1.0" ?>
 <robot xmlns:xacro="http://www.ros.org/wiki/xacro"  name="kumi">
-    <xacro:include filename="/home/andreas/dev_ws/src/kumi/description/xacro/variables.xacro" />
-    <xacro:include filename="/home/andreas/dev_ws/src/kumi/description/xacro/trajectory_control.xacro" />
-    <xacro:include filename="/home/andreas/dev_ws/src/kumi/description/xacro/kumi_mesh_stereocamera.xacro" />
-    <xacro:include filename="/home/andreas/dev_ws/src/kumi/description/xacro/sensors_config.xacro" />
+    <xacro:property name="kumi_share" value="$(find kumi)"/>
+    <xacro:include filename="${kumi_share}/description/xacro/variables.xacro" />
+    <xacro:include filename="${kumi_share}/description/xacro/trajectory_control.xacro" />
+    <xacro:include filename="${kumi_share}/description/xacro/kumi_mesh_stereocamera.xacro" />
+    <xacro:include filename="${kumi_share}/description/xacro/sensors_config.xacro" />
 </robot>

File: description/xacro/effort_control.xacro (robot description, xacro)
@@ -31,5 +31,5 @@
     <gazebo>
         <plugin filename="gz_ros2_control-system" name="gz_ros2_control::GazeboSimROS2ControlPlugin">
-            <parameters>/home/andreas/dev_ws/src/kumi/config/effort_control_config.yaml</parameters>
+            <parameters>$(find kumi)/config/effort_control_config.yaml</parameters>
         </plugin>
     </gazebo>

File: description/xacro/kumi_mesh_camera.xacro (robot description, xacro)
@@ -2,7 +2,8 @@
 <robot xmlns:xacro="http://www.ros.org/wiki/xacro" name="kumi">
     <xacro:property name="mesh_scale" value="0.001 0.001 0.001"/>
-    <xacro:property name="body_mesh" value="/home/andreas/dev_ws/src/kumi/description/mesh/body_v5.STL"/>
-    <xacro:property name="leg_mesh" value="/home/andreas/dev_ws/src/kumi/description/mesh/leg_v2.stl"/>
-    <xacro:property name="foot_mesh" value="/home/andreas/dev_ws/src/kumi/description/mesh/piedino_v3.STL"/>
+    <xacro:property name="mesh_dir" value="file://${kumi_share}/description/mesh"/>
+    <xacro:property name="body_mesh" value="${mesh_dir}/body_v5.STL"/>
+    <xacro:property name="leg_mesh" value="${mesh_dir}/leg_v2.stl"/>
+    <xacro:property name="foot_mesh" value="${mesh_dir}/piedino_v3.STL"/>
     <link name="body">
         <visual>

File: description/xacro/kumi_mesh_no_camera.xacro (robot description, xacro)
@@ -2,7 +2,8 @@
 <robot xmlns:xacro="http://www.ros.org/wiki/xacro" name="kumi">
     <xacro:property name="mesh_scale" value="0.001 0.001 0.001"/>
-    <xacro:property name="body_mesh" value="/home/andreas/dev_ws/src/kumi/description/mesh/body_v5.STL"/>
-    <xacro:property name="leg_mesh" value="/home/andreas/dev_ws/src/kumi/description/mesh/leg_v2.stl"/>
-    <xacro:property name="foot_mesh" value="/home/andreas/dev_ws/src/kumi/description/mesh/piedino_v3.STL"/>
+    <xacro:property name="mesh_dir" value="file://${kumi_share}/description/mesh"/>
+    <xacro:property name="body_mesh" value="${mesh_dir}/body_v5.STL"/>
+    <xacro:property name="leg_mesh" value="${mesh_dir}/leg_v2.stl"/>
+    <xacro:property name="foot_mesh" value="${mesh_dir}/piedino_v3.STL"/>
     <link name="body">
         <visual>
@@ -87,5 +88,5 @@
     <link name="front_foot">
         <visual>
-            <origin xyz="0 0 0" rpy="${pi/2} 0  ${-pi/2}"/>
+            <origin xyz="0 -0.007 0" rpy="${pi/2} 0  ${-pi/2}"/>
             <geometry>
                 <mesh filename="${foot_mesh}" scale="${mesh_scale}"/>
@@ -167,5 +168,5 @@
     <link name="rear_foot">
         <visual>
-            <origin xyz="0 0 0" rpy="${pi/2} 0  ${pi/2}"/>
+            <origin xyz="0 0.007 0" rpy="${pi/2} 0  ${pi/2}"/>
             <geometry>
                 <mesh filename="${foot_mesh}" scale="${mesh_scale}"/>

File: description/xacro/kumi_mesh_stereocamera.xacro (robot description, xacro)
@@ -2,8 +2,9 @@
 <robot xmlns:xacro="http://www.ros.org/wiki/xacro" name="kumi">
     <xacro:property name="mesh_scale" value="0.001 0.001 0.001"/>
-    <xacro:property name="body_mesh" value="/home/andreas/dev_ws/src/kumi/description/mesh/body_v5.STL"/>
-    <xacro:property name="leg_mesh" value="/home/andreas/dev_ws/src/kumi/description/mesh/leg_v2.stl"/>
-    <xacro:property name="foot_mesh" value="/home/andreas/dev_ws/src/kumi/description/mesh/piedino_v3.STL"/>
-    <xacro:property name="realsense_mesh" value="/home/andreas/dev_ws/src/kumi/description/mesh/realsense.stl"/>
+    <xacro:property name="mesh_dir" value="file://${kumi_share}/description/mesh"/>
+    <xacro:property name="body_mesh" value="${mesh_dir}/body_v5.STL"/>
+    <xacro:property name="leg_mesh" value="${mesh_dir}/leg_v2.stl"/>
+    <xacro:property name="foot_mesh" value="${mesh_dir}/piedino_v3.STL"/>
+    <xacro:property name="realsense_mesh" value="${mesh_dir}/realsense.stl"/>
     <link name="body">
         <visual>
@@ -144,13 +145,13 @@
         </sensor>
     </gazebo>
-    <joint name="front_ank" type="revolute">
+    <joint name="front_ank_y" type="revolute">
         <origin xyz="0 0 ${-leg_len}" rpy="0 0 0"/>
         <parent link="front_leg"/>
-        <child link="front_foot"/>
+        <child link="front_foot_dummy"/>
         <axis xyz="0 -1 0"/>
         <limit lower="${-2*pi}" upper="${2*pi}" velocity="5" effort="1000"/>
         <dynamics damping="0.1" friction="${joint_friction}"/>
     </joint>
-    <gazebo reference="front_ank">
+    <gazebo reference="front_ank_y">
         <sensor name="front_ank_force_torque" type="force_torque">
             <always_on>true</always_on>
@@ -162,7 +163,32 @@
         </sensor>
     </gazebo>
+    <link name="front_foot_dummy">
+        <inertial>
+            <origin xyz="0 0 0" rpy="0 0 0"/>
+            <mass value="0.001"/>
+            <inertia ixx="1e-5" ixy="0" ixz="0" iyy="1e-5" iyz="0" izz="1e-5"/>
+        </inertial>
+    </link>
+    <joint name="front_ank_z" type="revolute">
+        <origin xyz="0 0 0" rpy="0 0 0"/>
+        <parent link="front_foot_dummy"/>
+        <child link="front_foot"/>
+        <axis xyz="0 0 1"/>
+        <limit lower="${-0.1*pi}" upper="${0.1*pi}" velocity="5" effort="1000"/>
+        <dynamics damping="0.1" friction="${joint_friction}"/>
+    </joint>
+    <gazebo reference="front_ank_z">
+        <sensor name="front_ank_force_torque" type="force_torque">
+            <always_on>true</always_on>
+            <update_rate>500</update_rate>
+            <force_torque>
+                <frame>child</frame>
+                <measure_direction>child_to_parent</measure_direction>
+            </force_torque>
+        </sensor>
+    </gazebo>
     <link name="front_foot">
         <visual>
-            <origin xyz="0 0 0" rpy="${pi/2} 0  ${-pi/2}"/>
+            <origin xyz="0 -0.007 0" rpy="${pi/2} 0  ${-pi/2}"/>
             <geometry>
                 <mesh filename="${foot_mesh}" scale="${mesh_scale}"/>
@@ -172,5 +198,5 @@
             </material>
         </visual>
-        <collision>
+        <collision name="frontFootCollision">
             <origin xyz="0 0 0" rpy="${pi/2} 0  ${-pi/2}"/>
             <geometry>
@@ -224,13 +250,13 @@
         </inertial>
     </link>
-    <joint name="rear_ank" type="revolute">
+    <joint name="rear_ank_y" type="revolute">
         <origin xyz="0 0 ${-leg_len}" rpy="0 0 0"/>
         <parent link="rear_leg"/>
-        <child link="rear_foot"/>
+        <child link="rear_foot_dummy"/>
         <axis xyz="0 1 0"/>
         <limit lower="${-2*pi}" upper="${2*pi}" velocity="5" effort="1000"/>
         <dynamics damping="0.1" friction="${joint_friction}"/>
     </joint>
-    <gazebo reference="rear_ank">
+    <gazebo reference="rear_ank_y">
         <sensor name="rear_ank_force_torque" type="force_torque">
             <always_on>true</always_on>
@@ -242,7 +268,32 @@
         </sensor>
     </gazebo>
+    <link name="rear_foot_dummy">
+        <inertial>
+            <origin xyz="0 0 0" rpy="0 0 0"/>
+            <mass value="0.001"/>
+            <inertia ixx="1e-5" ixy="0" ixz="0" iyy="1e-5" iyz="0" izz="1e-5"/>
+        </inertial>
+    </link>
+    <joint name="rear_ank_z" type="revolute">
+        <origin xyz="0 0 0" rpy="0 0 0"/>
+        <parent link="rear_foot_dummy"/>
+        <child link="rear_foot"/>
+        <axis xyz="0 0 1"/>
+        <limit lower="${-0.1*pi}" upper="${0.1*pi}" velocity="5" effort="1000"/>
+        <dynamics damping="0.1" friction="${joint_friction}"/>
+    </joint>
+    <gazebo reference="rear_ank_z">
+        <sensor name="front_ank_force_torque" type="force_torque">
+            <always_on>true</always_on>
+            <update_rate>500</update_rate>
+            <force_torque>
+                <frame>child</frame>
+                <measure_direction>child_to_parent</measure_direction>
+            </force_torque>
+        </sensor>
+    </gazebo>
     <link name="rear_foot">
         <visual>
-            <origin xyz="0 0 0" rpy="${pi/2} 0  ${pi/2}"/>
+            <origin xyz="0 0.007 0" rpy="${pi/2} 0  ${pi/2}"/>
             <geometry>
                 <mesh filename="${foot_mesh}" scale="${mesh_scale}"/>
@@ -252,5 +303,5 @@
             </material>
         </visual>
-        <collision>
+        <collision name="rearFootCollision">
             <origin xyz="0 0 0" rpy="${pi/2} 0  ${pi/2}"/>
             <geometry>

File: description/xacro/sensors_config.xacro (robot description, xacro)
@@ -80,5 +80,5 @@
           <contact>
             <collision>frontFootCollision</collision>
-            <topic>/collisionFlag/rearFoot</topic>
+            <topic>/collisionFlag/frontFoot</topic>
           </contact>
           <always_on>1</always_on>

File: description/xacro/trajectory_control.xacro (robot description, xacro)
@@ -9,5 +9,10 @@
             <state_interface name="velocity"/>
         </joint>
-        <joint name="front_ank">
+        <joint name="front_ank_y">
+            <command_interface name="position"/>
+            <state_interface name="position"/>
+            <state_interface name="velocity"/>
+        </joint>
+        <joint name="front_ank_z">
             <command_interface name="position"/>
             <state_interface name="position"/>
@@ -19,5 +24,10 @@
             <state_interface name="velocity"/>
         </joint>
-        <joint name="rear_ank">
+        <joint name="rear_ank_y">
+            <command_interface name="position"/>
+            <state_interface name="position"/>
+            <state_interface name="velocity"/>
+        </joint>
+        <joint name="rear_ank_z">
             <command_interface name="position"/>
             <state_interface name="position"/>
@@ -27,5 +37,5 @@
     <gazebo>
         <plugin filename="gz_ros2_control-system" name="gz_ros2_control::GazeboSimROS2ControlPlugin">
-            <parameters>/home/andreas/dev_ws/src/kumi/config/trajectory_control_config.yaml</parameters>
+            <parameters>$(find kumi)/config/trajectory_control_config.yaml</parameters>
         </plugin>
     </gazebo>
