Commit message: mesh added, and world with stairs but still joint traj controller not working properly

File: description/xacro/controls.xacro (robot description, xacro)
@@ -5,9 +5,4 @@
         </hardware>
         <joint name="front_sh">
-            <command_interface name="position"/>
-            <state_interface name="position"/>
-            <state_interface name="velocity"/>
-        </joint>
-        <joint name="front_knee">
             <command_interface name="position"/>
             <state_interface name="position"/>
@@ -24,9 +19,4 @@
             <state_interface name="velocity"/>
         </joint>
-        <joint name="back_knee">
-            <command_interface name="position"/>
-            <state_interface name="position"/>
-            <state_interface name="velocity"/>
-        </joint>
         <joint name="back_ank">
             <command_interface name="position"/>
@@ -39,4 +29,7 @@
             <parameters>/home/andreas/dev_ws/install/kumi/share/kumi/config/kumi_control_config.yaml</parameters>
         </plugin>
+        <plugin name="gz::sim::systems::WrenchVisualizer" filename="gz-sim-wrench-visualizer-system">
+            <topic>/wrench</topic>
+        </plugin>
     </gazebo>
 </robot>

File: description/xacro/kumi_core.xacro (robot description, xacro)
@@ -84,5 +84,5 @@
     </link>
     <joint name="front_ank" type="revolute">
-        <origin xyz="0 0 ${-leg_len/2 - thikness/2}" rpy="0 0 0"/>
+        <origin xyz="0 0 ${-leg_len/4 - thikness/4}" rpy="0 0 0"/>
         <parent link="front_leg_d"/>
         <child link="front_foot"/>
@@ -93,5 +93,5 @@
     <link name="front_foot">
         <visual>
-            <origin xyz="0 0 0" rpy="0 0 0"/>
+            <origin xyz="0 0 ${-leg_len/4 - thikness/4}" rpy="0 0 0"/>
             <geometry>
                 <box size="${foot_len} ${foot_len} ${thikness/2}" />
@@ -102,5 +102,5 @@
         </visual>
         <collision>
-            <origin xyz="0 0 0" rpy="0 0 0"/>
+            <origin xyz="0 0 ${-leg_len/4 - thikness/4}" rpy="0 0 0"/>
             <geometry>
                 <box size="${foot_len-toll} ${foot_len-toll} ${thikness/2-toll}" />
@@ -108,5 +108,5 @@
         </collision>
         <inertial>
-            <origin xyz="0 0 0" rpy="0 0 0"/>
+            <origin xyz="0 0 ${-leg_len/4 - thikness/4}" rpy="0 0 0"/>
             <mass value="0.15" />
             <inertia ixx="0.001135" ixy="0.0" ixz="0.0" iyy="0.001135" iyz="0.0" izz="0.002083" />
@@ -174,5 +174,5 @@
     </link>
     <joint name="back_ank" type="revolute">
-        <origin xyz="0 0 ${-leg_len/2 - thikness/2}" rpy="0 0 0"/>
+        <origin xyz="0 0 ${-leg_len/4 - thikness/4}" rpy="0 0 0"/>
         <parent link="back_leg_d"/>
         <child link="back_foot"/>
@@ -183,5 +183,5 @@
     <link name="back_foot">
         <visual>
-            <origin xyz="0 0 0" rpy="0 0 0"/>
+            <origin xyz="0 0 ${-leg_len/4 - thikness/4}" rpy="0 0 0"/>
             <geometry>
                 <box size="${foot_len} ${foot_len} ${thikness/2}" />
@@ -192,5 +192,5 @@
         </visual>
         <collision>
-            <origin xyz="0 0 0" rpy="0 0 0"/>
+            <origin xyz="0 0 ${-leg_len/4 - thikness/4}" rpy="0 0 0"/>
             <geometry>
                 <box size="${foot_len-toll} ${foot_len-toll} ${thikness/2-toll}" />
@@ -198,5 +198,5 @@
         </collision>
         <inertial>
-            <origin xyz="0 0 0" rpy="0 0 0"/>
+            <origin xyz="0 0 ${-leg_len/4 - thikness/4}" rpy="0 0 0"/>
             <mass value="0.15" />
             <inertia ixx="0.001135" ixy="0.0" ixz="0.0" iyy="0.001135" iyz="0.0" izz="0.002083" />

File: description/xacro/variables.xacro (robot description, xacro)
@@ -5,6 +5,6 @@
     <xacro:property name="ang_up_lim" value="4" />
     <xacro:property name="thikness" value="0.15" />
-    <xacro:property name="lenght" value="0.5" />
-    <xacro:property name="leg_len" value="0.4" />
+    <xacro:property name="lenght" value="0.18" />
+    <xacro:property name="leg_len" value="0.11" />
     <xacro:property name="foot_len" value="0.5" />
     <xacro:property name="toll" value="0.005" />
