Commit message: added test_move node for PID tuning with foxglove

File: description/xacro/kumi_core.xacro (robot description, xacro)
@@ -27,5 +27,5 @@
         <parent link="body"/>
         <child link="front_leg"/>
-        <axis xyz="0 -1 0"/>
+        <axis xyz="0 1 0"/>
         <limit lower="-0.85" upper="${pi - 0.85}" velocity="5" effort="6"/>
         <dynamics damping="0.5" friction="${joint_friction}"/>
@@ -87,5 +87,5 @@
         <parent link="front_leg_d"/>
         <child link="front_foot"/>
-        <axis xyz="0 -1 0"/>
+        <axis xyz="0 1 0"/>
         <limit lower="-0.85" upper="0.85" velocity="5" effort="6"/>
         <dynamics damping="0.1" friction="${joint_friction}"/>
@@ -117,5 +117,5 @@
         <parent link="body"/>
         <child link="back_leg"/>
-        <axis xyz="0 -1 0"/>
+        <axis xyz="0 1 0"/>
         <limit lower="${-pi + 0.3}" upper="0.3" velocity="5" effort="6"/>
         <dynamics damping="0.1" friction="${joint_friction}"/>
@@ -177,5 +177,5 @@
         <parent link="back_leg_d"/>
         <child link="back_foot"/>
-        <axis xyz="0 -1 0"/>
+        <axis xyz="0 1 0"/>
         <limit lower="-0.85" upper="0.85" velocity="5" effort="6"/>
         <dynamics damping="0.1" friction="${joint_friction}"/>

File: description/xacro/kumi_mesh.xacro (robot description, xacro)
@@ -11,4 +11,7 @@
                 <mesh filename="${body_mesh}" scale="${mesh_scale}"/>
             </geometry>
+            <material name="gray">
+                <color rgba="0 0 0 0.8"/>
+            </material>
         </visual>
         <collision>
@@ -28,6 +31,6 @@
         <parent link="body"/>
         <child link="front_leg"/>
-        <axis xyz="0 1 0"/>
-        <limit lower="${-pi/4}" upper="${3*pi/4}" velocity="5" effort="1000"/>
+        <axis xyz="0 -1 0"/>
+        <limit lower="${-pi}" upper="${pi}" velocity="5" effort="1000"/>
         <dynamics damping="0.5" friction="${joint_friction}"/>
     </joint>
@@ -48,4 +51,7 @@
                 <mesh filename="${leg_mesh}" scale="${mesh_scale}"/>
             </geometry>
+            <material name="gray">
+                <color rgba="0 0 0 0.8"/>
+            </material>
         </visual>
         <collision>
@@ -65,6 +71,6 @@
         <parent link="front_leg"/>
         <child link="front_foot"/>
-        <axis xyz="0 1 0"/>
-        <limit lower="${-pi/2}" upper="${pi/2}" velocity="5" effort="1000"/>
+        <axis xyz="0 -1 0"/>
+        <limit lower="${-pi}" upper="${pi}" velocity="5" effort="1000"/>
         <dynamics damping="0.1" friction="${joint_friction}"/>
     </joint>
@@ -85,4 +91,7 @@
                 <mesh filename="${foot_mesh}" scale="${mesh_scale}"/>
             </geometry>
+            <material name="green">
+                <color rgba="0 1 0 0.8"/>
+            </material>
         </visual>
         <collision>
@@ -103,5 +112,5 @@
         <child link="back_leg"/>
         <axis xyz="0 -1 0"/>
-        <limit lower="${-pi/4}" upper="${3*pi/4}" velocity="5" effort="1000"/>
+        <limit lower="${-pi}" upper="${pi}" velocity="5" effort="1000"/>
         <dynamics damping="0.5" friction="${joint_friction}"/>
     </joint>
@@ -122,4 +131,7 @@
                 <mesh filename="${leg_mesh}" scale="${mesh_scale}"/>
             </geometry>
+            <material name="gray">
+                <color rgba="0 0 0 0.8"/>
+            </material>
         </visual>
         <collision>
@@ -140,5 +152,5 @@
         <child link="back_foot"/>
         <axis xyz="0 -1 0"/>
-        <limit lower="${-pi/2}" upper="${pi/2}" velocity="5" effort="1000"/>
+        <limit lower="${-pi}" upper="${pi}" velocity="5" effort="1000"/>
         <dynamics damping="0.1" friction="${joint_friction}"/>
     </joint>
@@ -159,4 +171,7 @@
                 <mesh filename="${foot_mesh}" scale="${mesh_scale}"/>
             </geometry>
+            <material name="red">
+                <color rgba="1 0 0 0.8"/>
+            </material>
         </visual>
         <collision>
