Commit message: trajectory control working well with simulated trajectories, PID tuning for effort controller is a work in progress. Nodes dedicated to bringup kumi, do a test move and reset the simulation working by receiving signals from MatLab script(only with the default empty world IDKY). Logging of the data from the topic /PID_data on matlab still not working good but at least exist. new file organization due to large file number. See you my self at the next commit

File: description/xacro/kumi_mesh.xacro (robot description, xacro)
@@ -32,5 +32,5 @@
         <child link="front_leg"/>
         <axis xyz="0 -1 0"/>
-        <limit lower="${-pi}" upper="${pi}" velocity="5" effort="1000"/>
+        <limit lower="${-2*pi}" upper="${2*pi}" velocity="5" effort="1000"/>
         <dynamics damping="0.5" friction="${joint_friction}"/>
     </joint>
@@ -72,5 +72,5 @@
         <child link="front_foot"/>
         <axis xyz="0 -1 0"/>
-        <limit lower="${-pi}" upper="${pi}" velocity="5" effort="1000"/>
+        <limit lower="${-2*pi}" upper="${2*pi}" velocity="5" effort="1000"/>
         <dynamics damping="0.1" friction="${joint_friction}"/>
     </joint>
@@ -111,6 +111,6 @@
         <parent link="body"/>
         <child link="back_leg"/>
-        <axis xyz="0 -1 0"/>
-        <limit lower="${-pi}" upper="${pi}" velocity="5" effort="1000"/>
+        <axis xyz="0 1 0"/>
+        <limit lower="${-2*pi}" upper="${2*pi}" velocity="5" effort="1000"/>
         <dynamics damping="0.5" friction="${joint_friction}"/>
     </joint>
@@ -151,6 +151,6 @@
         <parent link="back_leg"/>
         <child link="back_foot"/>
-        <axis xyz="0 -1 0"/>
-        <limit lower="${-pi}" upper="${pi}" velocity="5" effort="1000"/>
+        <axis xyz="0 1 0"/>
+        <limit lower="${-2*pi}" upper="${2*pi}" velocity="5" effort="1000"/>
         <dynamics damping="0.1" friction="${joint_friction}"/>
     </joint>

File: description/xacro/trajectory_control.xacro (robot description, xacro)
@@ -27,8 +27,5 @@
     <gazebo>
         <plugin filename="gz_ros2_control-system" name="gz_ros2_control::GazeboSimROS2ControlPlugin">
-            <parameters>/home/andreas/dev_ws/install/kumi/share/kumi/config/trajectory_control_config.yaml</parameters>
-        </plugin>
-        <plugin name="gz::sim::systems::WrenchVisualizer" filename="gz-sim-wrench-visualizer-system">
-            <topic>/wrench</topic>
+            <parameters>/home/andreas/dev_ws/src/kumi/config/trajectory_control_config.yaml</parameters>
         </plugin>
     </gazebo>

Commit message: pid controller updated to paratemter set from matlab, need to understand how to save the parameters after the reset

File: description/xacro/kumi_mesh.xacro (robot description, xacro)
@@ -118,7 +118,7 @@
         </visual>
         <collision name="frontFootCollision">
-            <origin xyz="0 0 0" rpy="${pi/2} 0  ${-pi/2}"/>
-            <geometry>
-                <mesh filename="${foot_mesh}" scale="${mesh_scale}"/>
+            <origin xyz="0 0 -0.023" rpy="0 0 0"/>
+            <geometry>
+                <box size="0.1 0.08 0.01" />
             </geometry>
         </collision>
@@ -220,7 +220,7 @@
         </visual>
         <collision name="rearFootCollision">
-            <origin xyz="0 0 0" rpy="${pi/2} 0  ${pi/2}"/>
-            <geometry>
-                <mesh filename="${foot_mesh}" scale="${mesh_scale}"/>
+            <origin xyz="0 0 -0.023" rpy="0 0 0"/>
+            <geometry>
+                <box size="0.1 0.08 0.01" />
             </geometry>
         </collision>

File: description/xacro/sensors_config.xacro (robot description, xacro)
@@ -7,5 +7,5 @@
             <visualize>true</visualize>
             <update_rate>30</update_rate>
-            <topic>frontCamera/image</topic>
+            <topic>/frontCamera/image</topic>
             <gz_frame_id>camera_rgb_frame</gz_frame_id>
             <camera name="intel_realsense_r200">
@@ -35,5 +35,5 @@
             <visualize>true</visualize>
             <update_rate>30</update_rate>
-            <topic>rearCamera/image</topic>
+            <topic>/rearCamera/image</topic>
             <gz_frame_id>camera_rgb_frame</gz_frame_id>
             <camera name="intel_realsense_r200">
@@ -77,8 +77,8 @@
     </gazebo>
     <gazebo reference="front_foot">
-        <sensor name='frontFootCollision' type='contact'>
+        <sensor name='frontFootCollisionSensor' type='contact'>
           <contact>
             <collision>frontFootCollision</collision>
-            <topic>/frontFootCollisionFlag</topic>
+            <topic>/collisionFlag/rearFoot</topic>
           </contact>
           <always_on>1</always_on>
@@ -87,8 +87,8 @@
     </gazebo>
     <gazebo reference="rear_foot">
-        <sensor name='rearFootCollision' type='contact'>
+        <sensor name='rearFootCollisionSensor' type='contact'>
           <contact>
             <collision>rearFootCollision</collision>
-            <topic>/rearFootCollisionFlag</topic>
+            <topic>/collisionFlag/rearFoot</topic>
           </contact>
           <always_on>1</always_on>
